Commit message: 添加imu

File: src/vehicle_description/urdf/diff_drive_robot.xacro (robot description, xacro)
@@ -32,5 +32,5 @@
       <child link="${name}_wheel"/>
       <origin xyz="${x_reflect * wheel_x} ${y_reflect * wheel_y} ${wheel_z}" rpy="${pi/2} 0 0"/>
-      <axis xyz="0 0 1"/>
+      <axis xyz="0 0 -1"/>
       <limit effort="50" velocity="20"/>
     </joint>

Commit message: feat: add Wi-Fi lidar hardware bringup

File: src/vehicle_description/urdf/diff_drive_robot.xacro (robot description, xacro)
@@ -112,60 +112,3 @@
     <origin xyz="0 0 ${pole_height/2 + 0.02}" rpy="0 0 0"/>
   </joint>
-  <!-- ===== Gazebo 颜色 ===== -->
-  <gazebo reference="base_link"><material>Gazebo/Blue</material></gazebo>
-  <gazebo reference="left_wheel"><material>Gazebo/DarkGrey</material></gazebo>
-  <gazebo reference="right_wheel"><material>Gazebo/DarkGrey</material></gazebo>
-  <gazebo reference="caster_link"><material>Gazebo/Grey</material></gazebo>
-  <gazebo reference="pole"><material>Gazebo/Black</material></gazebo>
-  <!-- ===== diff_drive 插件 ===== -->
-  <gazebo>
-    <plugin name="diff_drive" filename="libgazebo_ros_diff_drive.so">
-      <command_topic>/cmd_vel</command_topic>
-      <odometry_topic>/odom</odometry_topic>
-      <odometry_frame>odom</odometry_frame>
-      <robot_base_frame>base_footprint</robot_base_frame>
-      <left_joint>left_wheel_joint</left_joint>
-      <right_joint>right_wheel_joint</right_joint>
-      <wheel_separation>${2 * wheel_y}</wheel_separation>
-      <wheel_diameter>${2 * wheel_radius}</wheel_diameter>
-      <max_wheel_torque>20</max_wheel_torque>
-      <max_wheel_acceleration>5.0</max_wheel_acceleration>
-      <publish_odom>true</publish_odom>
-      <publish_odom_tf>true</publish_odom_tf>
-      <publish_wheel_tf>false</publish_wheel_tf>
-    </plugin>
-  </gazebo>
-  <!-- ===== LiDAR 传感器 ===== -->
-  <gazebo reference="lidar_link">
-    <sensor name="lidar" type="ray">
-      <pose>0 0 0 0 0 0</pose>
-      <visualize>false</visualize>
-      <update_rate>10</update_rate>
-      <ray>
-        <scan>
-          <horizontal>
-            <samples>720</samples>
-            <resolution>1</resolution>
-            <min_angle>-3.14159</min_angle>
-            <max_angle>3.14159</max_angle>
-          </horizontal>
-        </scan>
-        <range>
-          <min>0.3</min>
-          <max>80.0</max>
-          <resolution>0.01</resolution>
-        </range>
-        <noise>
-          <type>gaussian</type>
-          <mean>0.0</mean>
-          <stddev>0.01</stddev>
-        </noise>
-      </ray>
-      <plugin name="lidar_plugin" filename="libgazebo_ros_ray_sensor.so">
-        <remapping>~/out:=/scan</remapping>
-        <output_type>sensor_msgs/LaserScan</output_type>
-        <frame_name>lidar_link</frame_name>
-      </plugin>
-    </sensor>
-  </gazebo>
 </robot>

Commit message: feat: validate real robot USB lidar mapping

File: src/vehicle_description/urdf/diff_drive_robot.xacro (robot description, xacro)
@@ -1,5 +1,7 @@
 <?xml version="1.0"?>
 <robot xmlns:xacro="http://www.ros.org/wiki/xacro" name="diff_drive_robot">
-  <xacro:property name="wheel_radius" value="0.08"/>
+  <!-- 实车轮子直径 4 cm，左右轮中心距 13 cm。 -->
+  <xacro:property name="wheel_radius" value="0.02"/>
+  <xacro:property name="wheel_separation" value="0.13"/>
   <xacro:property name="wheel_width" value="0.04"/>
   <xacro:property name="body_length" value="0.4"/>
@@ -10,6 +12,6 @@
   <!-- 轮子放置：车身中偏后，左右对称 -->
   <xacro:property name="wheel_x" value="${-body_length/4}"/>
-  <xacro:property name="wheel_y" value="${body_width/2 + wheel_width/2 + 0.005}"/>
-  <xacro:property name="wheel_z" value="${-body_height/2 + wheel_radius  -0.05}"/>
+  <xacro:property name="wheel_y" value="${wheel_separation/2}"/>
+  <xacro:property name="wheel_z" value="${-body_height/2}"/>
   <xacro:property name="body_mass" value="10"/>
   <!-- ===== 轮子 macro ===== -->
@@ -41,5 +43,5 @@
     <parent link="base_footprint"/>
     <child link="base_link"/>
-    <origin xyz="0 0 ${wheel_radius + body_height/2 + 0.01}" rpy="0 0 0"/>
+    <origin xyz="0 0 ${wheel_radius + body_height/2}" rpy="0 0 0"/>
   </joint>
   <!-- ===== base_link ===== -->

File: src/vehicle_simulation/urdf/diff_drive_robot.gazebo.xacro (robot description, xacro)
@@ -18,5 +18,5 @@
       <left_joint>left_wheel_joint</left_joint>
       <right_joint>right_wheel_joint</right_joint>
-      <wheel_separation>${2 * wheel_y}</wheel_separation>
+      <wheel_separation>${wheel_separation}</wheel_separation>
       <wheel_diameter>${2 * wheel_radius}</wheel_diameter>
       <max_wheel_torque>20</max_wheel_torque>

Commit message: checkpoint: save real vehicle mapping state before IMU fusion

File: src/vehicle_description/urdf/diff_drive_robot.xacro (robot description, xacro)
@@ -1,10 +1,18 @@
 <?xml version="1.0"?>
 <robot xmlns:xacro="http://www.ros.org/wiki/xacro" name="diff_drive_robot">
-  <!-- 实车轮子直径 4 cm，左右轮中心距 13 cm。 -->
-  <xacro:property name="wheel_radius" value="0.02"/>
-  <xacro:property name="wheel_separation" value="0.13"/>
-  <xacro:property name="wheel_width" value="0.04"/>
-  <xacro:property name="body_length" value="0.4"/>
-  <xacro:property name="body_width" value="0.25"/>
+  <!-- 默认使用实车尺寸；Gazebo 可通过 Xacro 参数覆盖视觉/物理尺寸。 -->
+  <xacro:arg name="wheel_radius" default="0.02"/>
+  <xacro:arg name="wheel_separation" default="0.13"/>
+  <xacro:arg name="wheel_width" default="0.015"/>
+  <xacro:arg name="body_length" default="0.20"/>
+  <xacro:arg name="body_width" default="0.13"/>
+  <!-- 实车雷达相对车体 +X 顺时针约 37.5 度；仿真启动时覆盖为 0。 -->
+  <xacro:arg name="lidar_yaw" default="-0.654498469"/>
+  <xacro:property name="wheel_radius" value="$(arg wheel_radius)"/>
+  <xacro:property name="wheel_separation" value="$(arg wheel_separation)"/>
+  <xacro:property name="wheel_width" value="$(arg wheel_width)"/>
+  <xacro:property name="body_length" value="$(arg body_length)"/>
+  <xacro:property name="body_width" value="$(arg body_width)"/>
+  <xacro:property name="lidar_yaw" value="$(arg lidar_yaw)"/>
   <xacro:property name="body_height" value="0.08"/>
   <xacro:property name="caster_radius" value="0.03"/>
@@ -87,5 +95,5 @@
     <parent link="base_link"/>
     <child link="caster_link"/>
-    <origin xyz="${body_length/2 - 0.02} 0 ${-body_height/2 - caster_radius + 0.002}" rpy="0 0 0"/>
+    <origin xyz="${body_length/2 - 0.02} 0 ${caster_radius - wheel_radius - body_height/2}" rpy="0 0 0"/>
   </joint>
   <!-- ===== 支柱 + LiDAR ===== -->
@@ -112,5 +120,5 @@
     <parent link="pole"/>
     <child link="lidar_link"/>
-    <origin xyz="0 0 ${pole_height/2 + 0.02}" rpy="0 0 0"/>
+    <origin xyz="0 0 ${pole_height/2 + 0.02}" rpy="0 0 ${lidar_yaw}"/>
   </joint>
 </robot>
